File: knit_yarn.kicad_sch (KiCad schematic)
At the start: 10 parts, among them SW1 SW_SPST

Commit message: happy with graphics and added two more LEDs
Parts:
- added D5, D6: LED, LED_SMD:LED_0603_1608Metric_Pad1.05x0.95mm_HandSolder, symbol Device:LED
- added R5, R6: TBD, Resistor_SMD:R_0603_1608Metric_Pad0.98x0.95mm_HandSolder, symbol Device:R_US
Connections:
- net +3V0: now also SW1.2 (B), R5.1, R6.1; no longer BT1.1 (+)
- net GND: now also D5.1 (K), D6.1 (K)
- net at SW1.1 (A): now also BT1.1 (+)
- new net: D5.2 (A), R5.2
- new net: D6.2 (A), R6.2
Other:
- moved on the sheet: BT1, SW1
