File: knit_yarn_badge_v2/knit_yarn_badge_v2.kicad_sch (KiCad schematic)
At the start: 14 parts, among them SW1 SW_SPST

Commit message: non movable components locked
Parts:
- BT1: footprint Battery:BatteryHolder_MYOUNG_BS-07-A1BJ001_CR2032 -> Battery:BatteryHolder_Multicomp_BC-2001_1x2032
Changed lines of the file:
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@@
 			)
 		)
-		(property "Footprint" "Battery:BatteryHolder_MYOUNG_BS-07-A1BJ001_CR2032"
+		(property "Footprint" "Battery:BatteryHolder_Multicomp_BC-2001_1x2032"
 			(at 116.84 98.806 90)
 			(effects

Commit message: components arranged
Parts:
- BT1: footprint Battery:BatteryHolder_Multicomp_BC-2001_1x2032 -> Battery:BatteryHolder_Keystone_3002_1x2032
Changed lines of the file:
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@@
 			)
 		)
-		(property "Footprint" "Battery:BatteryHolder_Multicomp_BC-2001_1x2032"
+		(property "Footprint" "Battery:BatteryHolder_Keystone_3002_1x2032"
 			(at 116.84 98.806 90)
 			(effects
