File: knit_yarn_badge_v2/knit_yarn_badge_v2.kicad_pcb (KiCad board)
At the start: 2 copper layers, 33.8 x 36.1 mm, 14 parts, among them SW1 SW_SPST

Commit message: v2 ready for order
Routing:
- net Net-(D3-A): track 0.15 -> 9.89 mm
- net +3V0: track 49.0 -> 49.9 mm
Other:
- board text removed: "Stockholm, SWE"
